Commit message: Automated world generation and object placement

File: src/earthrover_vla_description/urdf/robot.xacro (robot description, xacro)
@@ -5,12 +5,12 @@
     <xacro:property name="pi_const" value="3.14159265" />
     <!-- Body Dimensions -->
-    <xacro:property name="a" value="1"/> <!-- Uses default gazebo units, m)-->
-    <xacro:property name="b" value="0.3"/>
-    <xacro:property name="c" value="1"/>
+    <xacro:property name="a" value="0.250"/> <!-- Uses default gazebo units, m)-->
+    <xacro:property name="b" value="0.160"/>
+    <xacro:property name="c" value="0.150"/>
     <!-- Wheel Dimensions -->
     <!-- Wheel radius-->
-    <xacro:property name="r" value="0.15" />
+    <xacro:property name="r" value="0.035" />
     <!-- wheel width -->
-    <xacro:property name="d" value="0.1" />
+    <xacro:property name="d" value="0.05" />
     <xacro:property name="s1" value="${b/2+r}"/>
     <xacro:property name="s2" value="${2*r}"/>
@@ -54,7 +54,7 @@
         <!-- Camera Dimensions and Properties -->
     <!-- Dimensions -->
-    <xacro:property name="cam_y" value="0.1" />
-    <xacro:property name="cam_z" value="0.1" />
-    <xacro:property name="cam_x" value="0.05" />
+    <xacro:property name="cam_y" value="0.06" />
+    <xacro:property name="cam_z" value="0.05" />
+    <xacro:property name="cam_x" value="0.03" />
     <!-- Mass-->
     <xacro:property name="cam_mass" value="${cam_y*cam_z*cam_x*d1}" />
